Commit message: retirar as " " porque estava a dar erro

File: p_g4_description/urdf/p_g4.gazebo.xacro (robot description, xacro)
@@ -52,4 +52,17 @@
     </sensor>
     <material>Gazebo/Grey</material>
+  </gazebo>
+  <gazebo reference="base_link">
+    <sensor name="base_link" type="contact">
+      <update_rate>1000.0</update_rate>
+      <always_on>true</always_on>
+      <contact>
+        <collision> base_footprint_fixed_joint_lump__base_link_collision</collision>
+      </contact>
+      <plugin name="base_link_contact_sensor_plugin" filename="libgazebo_ros_bumper.so">
+        <bumperTopicName>contact</bumperTopicName>
+        <frameName>world</frameName>
+      </plugin>
+    </sensor>
   </gazebo>
   <gazebo>
@@ -168,16 +181,3 @@
     </sensor>
   </gazebo>
-  <gazebo reference="base_link">
-    <sensor name="base_link" type="contact">
-      <update_rate>1000.0</update_rate>
-      <always_on>true</always_on>
-      <contact>
-        <collision> "base_footprint_fixed_joint_lump__base_link_collision" </collision>
-      </contact>
-      <plugin name="base_link_contact_sensor_plugin" filename="libgazebo_ros_bumper.so">
-        <bumperTopicName>contact</bumperTopicName>
-        <frameName>world</frameName>
-      </plugin>
-    </sensor>
-  </gazebo>
 </robot>

Commit message: arbitro funcional #5

File: p_g4_description/urdf/p_g4.gazebo.xacro (robot description, xacro)
@@ -181,3 +181,16 @@
     </sensor>
   </gazebo>
+  <gazebo reference="base_link">
+    <sensor name="base_link" type="contact">
+      <update_rate>1000.0</update_rate>
+      <always_on>true</always_on>
+      <contact>
+        <collision>base_footprint_fixed_joint_lump__base_link_collision</collision>
+      </contact>
+      <plugin name="base_link_contact_sensor_plugin" filename="libgazebo_ros_bumper.so">
+        <bumperTopicName>contact</bumperTopicName>
+        <frameName>world</frameName>
+      </plugin>
+    </sensor>
+  </gazebo>
 </robot>
