Commit message: update final #1

File: p_g4_description/urdf/properties.xacro (robot description, xacro)
@@ -8,7 +8,4 @@
     <material name="Orange">
         <color rgba="1.0 0.4 0.0 1.0"/>
-    </material>
-    <material name="sarascolor">
-        <color rgba="0.2 0.5 0.8 1.0"/>
     </material>
     <!--    Team hunt player colors-->
